Commit message: temp

File: jaka_description/urdf/jaka_swift.urdf (robot description, URDF)
Before this commit: robot jaka_zu5, 9 links, 8 joints
Links:
- link Link_0: geometry collision mesh filename=/home/buse/collaborice_ws/src/jaka_description/meshes/jaka_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; visual mesh filename=/home/buse/collaborice_ws/src/jaka_description/meshes/jaka_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
- link Link_1: geometry collision mesh filename=/home/buse/collaborice_ws/src/jaka_description/meshes/jaka_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; visual mesh filename=/home/buse/collaborice_ws/src/jaka_description/meshes/jaka_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
- link Link_2: geometry collision mesh filename=/home/buse/collaborice_ws/src/jaka_description/meshes/jaka_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; visual mesh filename=/home/buse/collaborice_ws/src/jaka_description/meshes/jaka_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
- link Link_3: geometry collision mesh filename=/home/buse/collaborice_ws/src/jaka_description/meshes/jaka_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; visual mesh filename=/home/buse/collaborice_ws/src/jaka_description/meshes/jaka_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
- link Link_4: geometry collision mesh filename=/home/buse/collaborice_ws/src/jaka_description/meshes/jaka_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; visual mesh filename=/home/buse/collaborice_ws/src/jaka_description/meshes/jaka_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
- link Link_5: geometry collision mesh filename=/home/buse/collaborice_ws/src/jaka_description/meshes/jaka_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; visual mesh filename=/home/buse/collaborice_ws/src/jaka_description/meshes/jaka_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
- link Link_6: geometry collision mesh filename=/home/buse/collaborice_ws/src/jaka_description/meshes/jaka_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; visual mesh filename=/home/buse/collaborice_ws/src/jaka_description/meshes/jaka_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
