Commit message: FIxed misc bugs

File: jaka_description/urdf/jaka.urdf (robot description, URDF)
Before this commit: robot jaka_zu5, 9 links, 8 joints
Joints:
- joint fixed: origin xyz=0 0 0 rpy=0 0 0.785 -> xyz=0 0 0 rpy=0 0 0

Commit message: Better launch structure

File: jaka_description/urdf/jaka.urdf (robot description, URDF)
Before this commit: robot jaka_zu5, 9 links, 8 joints
Joints:
- joint fixed: origin xyz=0 0 0 rpy=0 0 0 -> xyz=0 0 0 rpy=0 0 0.7854
